Commit message: Robot Material and Differential Pluggin

File: 07_GazeboSim/03_ConnectToRos2/01_robotMaterial.urdf (robot description, URDF)
Before this commit: robot robot, 4 links, 3 joints
Links:
- link link_chassis: geometry collision mesh filename=package://robot_description/meshes/chassis.stl; visual mesh filename=package://robot_description/meshes/chassis.stl
